Commit message: Implement tank turn mode, decoupled e-stop, SLAM tuning, and unified allrun pipeline

File: src/motor_control/urdf/robot.urdf (robot description, URDF)
Before this commit: robot mobile_robot, 7 links, 6 joints
Links:
- added link imu_link; visual box size=0.03 0.02 0.005
Joints:
- added joint base_imu_joint: type fixed, parent base_link, child imu_link, origin xyz=0.0 0.0 0.08 rpy=0 0 0
